File: WheelOfJoy.kicad_pcb (KiCad board)
At the start: 2 copper layers, 47.8 x 45.4 mm, 26 parts, among them CN1 JOY1, CN2 JOY2, CN3 JOY3, CN4 JOY4, CN5 DB15F, U1 74LS153, U2 74LS153, U3 74LS153

Commit message: Last port done
Routing:
- net Net-(CN1-Pad9): track 54.8 -> 53.4 mm, vias 6 -> 4
- net +5V: track 178.0 -> 177.1 mm
- net Net-(CN4-Pad1): track 38.9 -> 39.6 mm
- net GND: vias 6 -> 21
Other:
- board text added: "MINI :)"
- board text added: "V1"
- board text removed: "V2"

Commit message: Almost there
Parts:
- moved V3 0.41 mm to (146.3, 95.4)
- moved V5 0.13 mm to (165.7, 130.8)
Routing:
- net /d7: track 58.8 -> 64.0 mm, vias 3 -> 4
- net Net-(CN1-Pad9): track 53.4 -> 51.1 mm
- net +5V: track 177.1 -> 178.7 mm
- net Net-(CN4-Pad3): track 43.7 -> 42.4 mm
- net Net-(CN2-Pad9): track 44.4 -> 45.5 mm
- net Net-(CN2-Pad3): track 34.4 -> 35.4 mm
- net Net-(CN2-Pad4): track 30.1 -> 30.9 mm
- net Net-(CN4-Pad4): track 41.2 -> 41.8 mm
- net Net-(CN3-Pad4): track 45.2 -> 45.8 mm
- net GND: vias 21 -> 24

Commit message: YEAH!
Parts:
- C4: footprint Capacitor_SMD:C_1206_3216Metric_Pad1.33x1.80mm_HandSolder -> Capacitor_Tantalum_SMD:CP_EIA-7343-30_AVX-N_Pad2.25x2.55mm_HandSolder
- moved C4 0.89 mm to (156.7, 126.0)
Routing:
- net +5V: track 178.7 -> 174.7 mm, vias 21 -> 20
- net Net-(CN4-Pad3): track 42.4 -> 43.8 mm
- net Net-(CN4-Pad4): track 41.8 -> 42.8 mm
- net GND: vias 24 -> 23
